File: 4PCB.sch (KiCad schematic (older format))
At the start: 24 parts, among them SW1 SW_Push, U1 ATmega32U4-AU, Y1 16MHz

Commit message: Update 4PCB.sch
Connections:
- net COL2 is gone; now on net COL1: MX3.1 (COL), MX4.1 (COL)
- net COL1: no longer MX1.1 (COL), MX2.1 (COL)
- net ROW1: now also D2.1 (K), D4.1 (K); no longer D1.1 (K), D3.1 (K)
- new net COL0: MX1.1 (COL), MX2.1 (COL)
- new net ROW0: D1.1 (K), D3.1 (K)
Other:
- moved on the sheet: D1, D2, D3, D4
Changed lines of the file:
@@
 EESchema Schematic File Version 4
+LIBS:75PCB-cache
 EELAYER 30 0
 EELAYER END
@@
 $EndComp
 Text GLabel 8750 3150 1    50   Input ~ 0
-COL2
+COL1
 Text GLabel 7750 3150 1    50   Input ~ 0
-COL1
-Wire Wire Line
-	7150 4850 8500 4850
-Text GLabel 7150 4850 0    50   Input ~ 0
-ROW2
-Text GLabel 7150 4000 0    50   Input ~ 0
+COL0
+Text GLabel 7150 4950 0    50   Input ~ 0
 ROW1
-Wire Wire Line
-	7500 4000 8500 4000
-Connection ~ 7500 4000
-Wire Wire Line
-	7150 4000 7500 4000
+Text GLabel 7150 3950 0    50   Input ~ 0
+ROW0
 Wire Wire Line
 	8750 3550 8750 4550
@@
 Wire Wire Line
 	7750 3150 7750 3550
-Wire Wire Line
-	8500 3750 8550 3750
-Wire Wire Line
-	8500 3800 8500 3750
-Wire Wire Line
-	7500 4750 7550 4750
-Wire Wire Line
-	7500 4800 7500 4750
-Wire Wire Line
-	8500 4750 8550 4750
-Wire Wire Line
-	8500 4800 8500 4750
 $Comp
 L Device:D_Small D4
 U 1 1 5F669C0B
-P 8500 4900
-F 0 "D4" V 8546 4832 50  0000 R CNN
-F 1 "D_Small" V 8455 4832 50  0000 R CNN
-F 2 "Diode_SMD:D_SOD-123" V 8500 4900 50  0001 C CNN
-F 3 "~" V 8500 4900 50  0001 C CNN
-	1    8500 4900
+P 8450 4850
+F 0 "D4" V 8496 4782 50  0000 R CNN
+F 1 "D_Small" V 8405 4782 50  0000 R CNN
+F 2 "Diode_SMD:D_SOD-123" V 8450 4850 50  0001 C CNN
+F 3 "~" V 8450 4850 50  0001 C CNN
+	1    8450 4850
 	0    -1   -1   0
 $EndComp
@@
 L Device:D_Small D2
 U 1 1 5F669796
-P 7500 4900
-F 0 "D2" V 7546 4832 50  0000 R CNN
-F 1 "D_Small" V 7455 4832 50  0000 R CNN
-F 2 "Diode_SMD:D_SOD-123" V 7500 4900 50  0001 C CNN
-F 3 "~" V 7500 4900 50  0001 C CNN
-	1    7500 4900
+P 7450 4850
+F 0 "D2" V 7496 4782 50  0000 R CNN
+F 1 "D_Small" V 7405 4782 50  0000 R CNN
+F 2 "Diode_SMD:D_SOD-123" V 7450 4850 50  0001 C CNN
+F 3 "~" V 7450 4850 50  0001 C CNN
+	1    7450 4850
 	0    -1   -1   0
 $EndComp
@@
 L Device:D_Small D3
 U 1 1 5F668CE6
-P 8500 3900
-F 0 "D3" V 8546 3832 50  0000 R CNN
-F 1 "D_Small" V 8455 3832 50  0000 R CNN
-F 2 "Diode_SMD:D_SOD-123" V 8500 3900 50  0001 C CNN
-F 3 "~" V 8500 3900 50  0001 C CNN
-	1    8500 3900
+P 8450 3850
+F 0 "D3" V 8496 3782 50  0000 R CNN
+F 1 "D_Small" V 8405 3782 50  0000 R CNN
+F 2 "Diode_SMD:D_SOD-123" V 8450 3850 50  0001 C CNN
+F 3 "~" V 8450 3850 50  0001 C CNN
+	1    8450 3850
 	0    -1   -1   0
 $EndComp
@@
 	1    0    0    -1
 $EndComp
-Wire Wire Line
-	7500 3750 7500 3800
-Wire Wire Line
-	7550 3750 7500 3750
 $Comp
 L Device:D_Small D1
 U 1 1 5F65FB74
-P 7500 3900
-F 0 "D1" V 7546 3832 50  0000 R CNN
-F 1 "D_Small" V 7455 3832 50  0000 R CNN
-F 2 "Diode_SMD:D_SOD-123" V 7500 3900 50  0001 C CNN
-F 3 "~" V 7500 3900 50  0001 C CNN
-	1    7500 3900
+P 7450 3850
+F 0 "D1" V 7496 3782 50  0000 R CNN
+F 1 "D_Small" V 7405 3782 50  0000 R CNN
+F 2 "Diode_SMD:D_SOD-123" V 7450 3850 50  0001 C CNN
+F 3 "~" V 7450 3850 50  0001 C CNN
+	1    7450 3850
 	0    -1   -1   0
 $EndComp
@@
 	1    0    0    -1
 $EndComp
+Wire Wire Line
+	8550 3750 8450 3750
+Wire Wire Line
+	7550 3750 7450 3750
+Wire Wire Line
+	7550 4750 7450 4750
+Wire Wire Line
+	8550 4750 8450 4750
+Wire Wire Line
+	7150 3950 7450 3950
+Connection ~ 7450 3950
+Wire Wire Line
+	7450 3950 8450 3950
+Wire Wire Line
+	7150 4950 7450 4950
+Wire Wire Line
+	7450 4950 8450 4950
+Connection ~ 7450 4950
 $EndSCHEMATC
